File: japanese-connection.kicad_pcb (KiCad board)
At the start: 2 copper layers, 82 x 52 mm, 9 parts, among them J1 Conn_01x06, J5 Conn_01x06, U1 ProMicro

Commit message: feat: retraced, matches Cheapino
It should now be possible to hook a cheapino to this build, with some
changes to the firmware of course.
Parts:
- renumbered left to left1, right to right1
Connections:
- J5 pad 1: Net-(J5-Pin_1) -> row5
- U1 pad 7: Net-(J5-Pin_1) -> row5
- left1 pad 1: GND -> l_col1
- left1 pad 2: l_col3 -> l_col2
- left1 pad 3: row2 -> l_col3
- left1 pad 4: l_col2 -> row4
- left1 pad 5: row1 -> row3
- left1 pad 6: l_col1 -> row2
- left1 pad 7: row4 -> row1
- left1 pad 8: row3 -> row5
- right1 pad 1: row1 -> r_col1
- right1 pad 2: r_col1 -> r_col2
- right1 pad 3: row2 -> r_col3
- right1 pad 4: r_col2 -> row5
- right1 pad 5: row3 -> row1
- right1 pad 6: r_col3 -> row2
- right1 pad 7: row4 -> row3
- right1 pad 8: GND -> row4
Routing:
- net row5: track 0.00 -> 83.1 mm, vias 0 -> 2
- net GND: track 67.3 -> 10.6 mm
- net r_col3: track 20.8 -> 38.4 mm
- net r_col2: track 20.8 -> 37.0 mm
- net row2: track 79.7 -> 65.5 mm, vias 0 -> 1
- net Net-(J5-Pin_1): track 10.7 -> 0.00 mm
- net row4: track 78.6 -> 69.9 mm, vias 0 -> 1
- net l_col2: track 21.1 -> 27.1 mm
- net l_col1: track 21.1 -> 26.2 mm
- net row1: track 71.2 -> 75.1 mm
- net row3: track 71.0 -> 67.3 mm
- net r_col1: track 20.8 -> 23.9 mm
- net l_col3: track 21.1 -> 23.5 mm
- added copper zone on B.Cu, net GND
- added copper zone on F.Cu, net GND
- removed copper zone on B.Cu, net (none)
- removed copper zone on F.Cu, net (none)
Other:
- board text added: "The Japanese Connection"
