File: japanese-connection.kicad_sch (KiCad schematic)
At the start: 5 parts, among them J1 Conn_01x06, J5 Conn_01x06, U1 ProMicro

Commit message: feat: retraced, matches Cheapino
It should now be possible to hook a cheapino to this build, with some
changes to the firmware of course.
Connections:
- net GND: no longer left1.1, right1.8
- net l_col1: now also left1.1; no longer left1.6
- net l_col2: now also left1.2; no longer left1.4
- net l_col3: now also left1.3; no longer left1.2
- net r_col1: now also right1.1; no longer right1.2
- net r_col2: now also right1.2; no longer right1.4
- net r_col3: now also right1.3; no longer right1.6
- net row1: now also left1.7, right1.5; no longer left1.5, right1.1
- net row2: now also left1.6, right1.6; no longer left1.3, right1.3
- net row3: now also left1.5, right1.7; no longer left1.8, right1.5
- net row4: now also left1.4, right1.8; no longer left1.7, right1.7
- net row5: now reaches J5.1 (Pin_1), U1.7 (4/D4)
- net row5: now also left1.8, right1.4
